File: Hardware/ledmatrix.brd (EAGLE design)
At the start: 160 x 100 mm, 86 parts, among them T1 2N2222, T2 2N2222, T3 2N2222, T4 2N2222, T5 2N2222, T6 2N2222

Commit message: eagle restart
Parts:
- removed T2, T3, T4, T5, T6: 2N2222, transistor:TO18
Connections:
- new net N$3: LED11.K, LED14.K, LED35.K, LED38.K, LED59.K, LED62.K
- net COL12: no longer LED61.K
- net N$1: now also LED12.K, LED13.K, LED36.K, LED37.K, LED61.K, T1.3; no longer LED61.A
Changed lines of the file:
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@@
 <element name="LED72" library="led" package="LED5MM" value="" x="-48.26" y="72.39"/>
 <element name="T1" library="transistor" package="TO18" value="2N2222" x="-22.86" y="86.36"/>
-<element name="T2" library="transistor" package="TO18" value="2N2222" x="-38.1" y="86.36"/>
-<element name="T3" library="transistor" package="TO18" value="2N2222" x="-53.34" y="86.36"/>
-<element name="T4" library="transistor" package="TO18" value="2N2222" x="-68.58" y="86.36"/>
-<element name="T5" library="transistor" package="TO18" value="2N2222" x="-83.82" y="86.36"/>
-<element name="T6" library="transistor" package="TO18" value="2N2222" x="-22.86" y="92.71"/>
 <element name="R1" library="eagle-ltspice" package="0204/7" value="" x="-31.75" y="91.44">
 <attribute name="SPICEMODEL" value="NONE" x="0" y="0" size="1.778" layer="27" display="off"/>
@@
 <signal name="COL12">
 <contactref element="SV2" pad="12"/>
-<contactref element="LED61" pad="K"/>
-<wire x1="31.75" y1="5.08" x2="-85.09" y2="57.15" width="0" layer="19" extent="1-1"/>
 </signal>
 <signal name="N$2">
@@
 </signal>
 <signal name="N$1">
-<contactref element="LED61" pad="A"/>
+<contactref element="LED61" pad="K"/>
 <contactref element="LED60" pad="K"/>
-<wire x1="-72.39" y1="57.15" x2="-87.63" y2="57.15" width="0" layer="19" extent="1-1"/>
+<contactref element="LED37" pad="K"/>
+<contactref element="LED12" pad="K"/>
+<contactref element="LED13" pad="K"/>
+<contactref element="LED36" pad="K"/>
+<contactref element="T1" pad="3"/>
+<wire x1="-85.09" y1="3.81" x2="-97.79" y2="3.81" width="0" layer="19" extent="1-1"/>
+<wire x1="-46.99" y1="34.29" x2="-85.09" y2="3.81" width="0" layer="19" extent="1-1"/>
+<wire x1="-34.29" y1="34.29" x2="-46.99" y2="34.29" width="0" layer="19" extent="1-1"/>
+<wire x1="-72.39" y1="57.15" x2="-46.99" y2="34.29" width="0" layer="19" extent="1-1"/>
+<wire x1="-85.09" y1="57.15" x2="-72.39" y2="57.15" width="0" layer="19" extent="1-1"/>
+<wire x1="-21.59" y1="87.63" x2="-34.29" y2="34.29" width="0" layer="19" extent="1-1"/>
+</signal>
+<signal name="N$3">
+<contactref element="LED62" pad="K"/>
+<contactref element="LED59" pad="K"/>
+<contactref element="LED38" pad="K"/>
+<contactref element="LED11" pad="K"/>
+<contactref element="LED14" pad="K"/>
+<contactref element="LED35" pad="K"/>
+<wire x1="-59.69" y1="57.15" x2="-97.79" y2="57.15" width="0" layer="19" extent="1-1"/>
+<wire x1="-59.69" y1="72.39" x2="-59.69" y2="57.15" width="0" layer="19" extent="1-1"/>
+<wire x1="-59.69" y1="34.29" x2="-59.69" y2="57.15" width="0" layer="19" extent="1-1"/>
+<wire x1="-21.59" y1="34.29" x2="-59.69" y2="34.29" width="0" layer="19" extent="1-1"/>
+<wire x1="-21.59" y1="11.43" x2="-21.59" y2="34.29" width="0" layer="19" extent="1-1"/>
 </signal>
 </signals>
