File: Hardware/eagle/untitled.brd (EAGLE design)
At the start: 252.7 x 100 mm, 86 parts, among them T1 2N2222, T2 2N2222, T3 2N2222, T4 2N2222, T5 2N2222, T6 2N2222

Commit message: with matrix
Parts:
- LED1, LED10, LED11, LED12, LED13, LED14, LED15, LED16, LED17, LED18, LED19, LED2, LED20, LED21, LED22, LED23, LED24, LED25, LED26, LED27, LED28, LED29, LED3, LED30, LED31, LED32, LED33, LED34, LED35, LED36, LED37, LED38, LED39, LED4, LED40, LED41, LED42, LED43, LED44, LED45, LED46, LED47, LED48, LED49, LED5, LED50, LED51, LED52, LED53, LED54, LED55, LED56, LED57, LED58, LED59, LED6, LED60, LED61, LED62, LED63, LED64, LED65, LED66, LED67, LED68, LED69, LED7, LED70, LED71, LED72, LED8, LED9: device eagle-ltspice:LED_LD260 -> led:LED5MM
- R1, R2, R3, R4, R5, R6: device resistor:0411/15 -> rcl:0207/10
- moved R6 172.2 mm to (6.35, -29.2), turned to 0 degrees
- moved R1 156.2 mm to (6.35, -3.81)
- moved R4 148.5 mm to (6.35, -19.1)
- moved R5 134.8 mm to (6.35, -24.1)
- moved T5 128.7 mm to (193.0, 7.62)
- moved R3 65.6 mm to (6.35, -14.0)
- moved R2 63.9 mm to (6.35, -8.89)
- moved T6 63.2 mm to (160.0, 5.08)
- moved T2 22.5 mm to (194.3, 66.0)
- moved T3 13.7 mm to (198.1, 36.8)
- moved T4 9.67 mm to (193.0, 16.5)
- moved T1 4.02 mm to (186.7, 76.2)
- moved LED58 1.80 mm to (115.6, 58.4), turned to 45 degrees
- turned LED1 to 45 degrees
- turned LED10 to 45 degrees
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Connections:
- new net N$10: LED16.K, LED21.K, LED28.K, LED33.K, LED39.K, LED4.K, LED45.K, LED51.K, LED57.K, LED63.K, LED69.K, LED9.K
- new net N$2: LED1.K, LED12.K, LED13.K, LED24.K, LED25.K, LED36.K, LED42.K, LED48.K, LED54.K, LED60.K, LED66.K, LED72.K, R1.1
- new net N$24: LED17.K, LED20.K, LED29.K, LED32.K, LED38.K, LED44.K, LED5.K, LED50.K, LED56.K, LED62.K, LED68.K, LED8.K, R5.1
- new net N$25: R4.2
- new net N$26: SV2.2, T1.2
- new net N$27: LED18.K, LED19.K, LED30.K, LED31.K, LED37.K, LED43.K, LED49.K, LED55.K, LED6.K, LED61.K, LED67.K, LED7.K, R6.1
- new net N$28: SV2.3, T2.2
- new net N$29: SV2.4, T3.2
- new net N$30: SV2.5, T4.2
- new net N$31: SV2.6, T5.2
- new net N$32: SV2.7, T6.2
- new net N$4: R2.2, T2.3
- new net N$7: LED10.K, LED15.K, LED22.K, LED27.K, LED3.K, LED34.K, LED40.K, LED46.K, LED52.K, LED58.K, LED64.K, LED70.K, R3.1
- net N$11: now also LED10.A, LED11.A, LED7.A, LED8.A, LED9.A
- net N$12: now also LED14.A, LED15.A, LED16.A, LED17.A, LED18.A
- net N$13: now also LED19.A, LED20.A, LED21.A, LED22.A, LED23.A
- net N$14: now also LED26.A, LED27.A, LED28.A, LED29.A, LED30.A
- net N$15: now also LED31.A, LED32.A, LED33.A, LED34.A, LED35.A
- net N$16: now also LED37.A, LED38.A, LED39.A, LED40.A, LED41.A
- net N$17: now also LED43.A, LED44.A, LED45.A, LED46.A, LED47.A
- net N$18: now also LED49.A, LED50.A, LED51.A, LED52.A, LED53.A
- net N$19: now also LED55.A, LED56.A, LED57.A, LED58.A, LED59.A
- net N$20: now also LED61.A, LED62.A, LED63.A, LED64.A, LED65.A
- net N$21: now also LED67.A, LED68.A, LED69.A, LED70.A, LED71.A
- net N$23: now also LED2.A, LED3.A, LED4.A, LED5.A, LED6.A
- net N$3: now also LED11.K, LED14.K, LED2.K, LED23.K, LED26.K, LED35.K, LED41.K, LED47.K, LED53.K, LED59.K, LED65.K, LED71.K, R2.1; no longer T2.3
- net N$6: no longer R4.1, R4.2
- net N$9: now also R6.2; no longer R6.1

Commit message: working
Parts:
- added R10, R11, R12, R13, R7, R9: (no value), rcl:0207/10
- SV1: device con-lsta:FE12 -> con-lstb:MA12-1
- SV2: device con-lsta:FE08 -> con-lstb:MA07-1
- moved R1 116.5 mm to (99.6, 66.0), turned to 180 degrees
- moved LED72 115.1 mm to (245.6, 66.0), turned to 225 degrees
- moved LED63 114.1 mm to (234.4, 31.8), turned to 225 degrees
- moved LED71 114.0 mm to (245.3, 54.6), turned to 225 degrees
- moved LED69 114.0 mm to (245.7, 31.8), turned to 225 degrees
- moved LED70 113.6 mm to (245.5, 43.2), turned to 225 degrees
- moved LED66 113.0 mm to (234.6, 66.5), turned to 225 degrees
- moved R2 112.9 mm to (99.8, 54.4), turned to 180 degrees
- moved LED68 112.7 mm to (245.7, 21.2), turned to 225 degrees
- moved LED67 112.7 mm to (245.6, 10.8), turned to 225 degrees
- moved LED61 112.5 mm to (234.2, 10.9), turned to 225 degrees
- moved LED64 112.5 mm to (234.3, 43.3), turned to 225 degrees
- moved LED62 112.4 mm to (234.0, 21.7), turned to 225 degrees
- moved LED65 112.4 mm to (234.6, 54.0), turned to 225 degrees
- moved T3 111.0 mm to (87.3, 43.6), turned to 180 degrees
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Connections:
- new net N$33: R11.1, T4.2
- new net N$34: R13.2, SV2.7
- new net N$35: R10.1, T3.2
- new net N$36: R12.1, T5.2
- new net N$37: R13.1, T6.2
- net N$10: now also R4.1
- net N$25: now also R7.1, T1.2; no longer R4.2
- net N$26: now also R7.2; no longer T1.2
- net N$28: now also R9.1; no longer SV2.3
- net N$29: now also R9.2, SV2.3; no longer SV2.4, T3.2
- net N$30: now also R10.2, SV2.4; no longer SV2.5, T4.2
- net N$31: now also R11.2, SV2.5; no longer SV2.6, T5.2
- net N$32: now also R12.2, SV2.6; no longer SV2.7, T6.2
- net N$6: now also R4.2
Routing:
- net N$22: track 0.00 -> 193.3 mm
- net N$21: track 0.00 -> 172.9 mm
- net N$20: track 0.00 -> 165.5 mm
- net N$19: track 0.00 -> 153.8 mm
- net N$18: track 0.00 -> 142.5 mm
- net N$24: track 0.00 -> 141.5 mm
- net N$10: track 0.00 -> 140.8 mm
- net N$2: track 0.00 -> 140.7 mm
- net N$3: track 0.00 -> 140.3 mm
- net N$7: track 0.00 -> 140.1 mm
- net N$27: track 0.00 -> 139.7 mm
- net N$17: track 0.00 -> 133.2 mm
- net N$16: track 0.00 -> 124.4 mm
- net N$15: track 0.00 -> 113.4 mm
- net N$14: track 0.00 -> 102.1 mm
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Other:
- board size 252.7 x 100 mm -> 197.5 x 86 mm
