File: Hardware/eagle/untitled.sch (EAGLE design)
At the start: 86 parts, among them T1 2N2222, T2 2N2222, T3 2N2222, T4 2N2222, T5 2N2222, T6 2N2222

Commit message: with matrix
Parts:
- LED1, LED10, LED11, LED12, LED13, LED14, LED15, LED16, LED17, LED18, LED19, LED2, LED20, LED21, LED22, LED23, LED24, LED25, LED26, LED27, LED28, LED29, LED3, LED30, LED31, LED32, LED33, LED34, LED35, LED36, LED37, LED38, LED39, LED4, LED40, LED41, LED42, LED43, LED44, LED45, LED46, LED47, LED48, LED49, LED5, LED50, LED51, LED52, LED53, LED54, LED55, LED56, LED57, LED58, LED59, LED6, LED60, LED61, LED62, LED63, LED64, LED65, LED66, LED67, LED68, LED69, LED7, LED70, LED71, LED72, LED8, LED9: device eagle-ltspice:LED_ELD260 -> led:LED5MM
- R1, R2, R3, R4, R5, R6: device resistor:R-EU_0411/15 -> rcl:R-EU_0207/10
Connections:
- new net N$10: LED16.C, LED21.C, LED28.C, LED33.C, LED39.C, LED4.C, LED45.C, LED51.C, LED57.C, LED63.C, LED69.C, LED9.C
- new net N$2: LED1.C, LED12.C, LED13.C, LED24.C, LED25.C, LED36.C, LED42.C, LED48.C, LED54.C, LED60.C, LED66.C, LED72.C, R1.1
- new net N$24: LED17.C, LED20.C, LED29.C, LED32.C, LED38.C, LED44.C, LED5.C, LED50.C, LED56.C, LED62.C, LED68.C, LED8.C, R5.1
- new net N$25: R4.2
- new net N$26: SV2.2, T1.B
- new net N$27: LED18.C, LED19.C, LED30.C, LED31.C, LED37.C, LED43.C, LED49.C, LED55.C, LED6.C, LED61.C, LED67.C, LED7.C, R6.1
- new net N$28: SV2.3, T2.B
- new net N$29: SV2.4, T3.B
- new net N$30: SV2.5, T4.B
- new net N$31: SV2.6, T5.B
- new net N$32: SV2.7, T6.B
- new net N$4: R2.2, T2.C
- new net N$7: LED10.C, LED15.C, LED22.C, LED27.C, LED3.C, LED34.C, LED40.C, LED46.C, LED52.C, LED58.C, LED64.C, LED70.C, R3.1
- net N$11: now also LED10.A, LED11.A, LED7.A, LED8.A, LED9.A
- net N$12: now also LED14.A, LED15.A, LED16.A, LED17.A, LED18.A
- net N$13: now also LED19.A, LED20.A, LED21.A, LED22.A, LED23.A
- net N$14: now also LED26.A, LED27.A, LED28.A, LED29.A, LED30.A
- net N$15: now also LED31.A, LED32.A, LED33.A, LED34.A, LED35.A
- net N$16: now also LED37.A, LED38.A, LED39.A, LED40.A, LED41.A
- net N$17: now also LED43.A, LED44.A, LED45.A, LED46.A, LED47.A
- net N$18: now also LED49.A, LED50.A, LED51.A, LED52.A, LED53.A
- net N$19: now also LED55.A, LED56.A, LED57.A, LED58.A, LED59.A
- net N$20: now also LED61.A, LED62.A, LED63.A, LED64.A, LED65.A
- net N$21: now also LED67.A, LED68.A, LED69.A, LED70.A, LED71.A
- net N$23: now also LED2.A, LED3.A, LED4.A, LED5.A, LED6.A
- net N$3: now also LED11.C, LED14.C, LED2.C, LED23.C, LED26.C, LED35.C, LED41.C, LED47.C, LED53.C, LED59.C, LED65.C, LED71.C, R2.1; no longer T2.C
- net N$6: no longer R4.1, R4.2
- net N$9: now also R6.2; no longer R6.1
Other:
- moved on the sheet: R1, R2, R3, R4, R5, R6, SV2

Commit message: working
Parts:
- added R10, R11, R12, R13, R7, R9: (no value), rcl:R-EU_0207/10
- SV1: device con-lsta:FE12-1 -> con-lstb:MA12-1
- SV2: device con-lsta:FE08-1 -> con-lstb:MA07-1
Connections:
- new net N$33: R11.1, T4.B
- new net N$34: R13.2, SV2.7
- new net N$35: R10.1, T3.B
- new net N$36: R12.1, T5.B
- new net N$37: R13.1, T6.B
- net N$10: now also R4.1
- net N$25: now also R7.1, T1.B; no longer R4.2
- net N$26: now also R7.2; no longer T1.B
- net N$28: now also R9.1; no longer SV2.3
- net N$29: now also R9.2, SV2.3; no longer SV2.4, T3.B
- net N$30: now also R10.2, SV2.4; no longer SV2.5, T4.B
- net N$31: now also R11.2, SV2.5; no longer SV2.6, T5.B
- net N$32: now also R12.2, SV2.6; no longer SV2.7, T6.B
- net N$6: now also R4.2
